File: lowprofile-pcb/Pteron36v0.kicad_pcb (KiCad board)
At the start: 2 copper layers, 123.5 x 95.6 mm, 47 parts, among them J1 AudioJack4, J2 AudioJack4, SW1 SW_PUSH, SW10 SW_PUSH, SW12 SW_PUSH, SW13 SW_PUSH, SW14 SW_PUSH, SW15 SW_PUSH, SW17 SW_PUSH, SW18 SW_PUSH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

Commit message: added custom anime silk layer
Parts:
- removed LOGO3, LOGO4: LOGO-OTL, personal-logo:peacock-medium
- added ?: , Anime_Lib:anime_girl_vertical_2, F.Cu at (124.5, 96.5)
