File: lowprofile-pcb/Pteron36v0_bikini_girl.kicad_pcb (KiCad board)
At the start: 2 copper layers, 123.5 x 95.6 mm, 46 parts, among them J1 AudioJack4, J2 AudioJack4, SW1 SW_PUSH, SW10 SW_PUSH, SW12 SW_PUSH, SW13 SW_PUSH, SW14 SW_PUSH, SW15 SW_PUSH, SW17 SW_PUSH, SW18 SW_PUSH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

Commit message: added bikini picture, fixed bad lines on old anime pic
Parts:
- removed the ? at (124.5, 94.0)
- added ?: , Anime_Lib:anime_bikini_girl, B.Cu at (127.0, 96.5)
